File: hardware/central-unit-hub/central-unit-hub.kicad_sch (KiCad schematic)
At the start: 6 parts, among them U2 ESP32-S3-WROOM-1, U3 MDBT50Q-1MV2, U4 BQ24074RGT

Commit message: v1.5: Minor Fixes
Parts:
- removed U2: ESP32-S3-WROOM-1, RF_Module:ESP32-S3-WROOM-1, symbol RF_Module:ESP32-S3-WROOM-1
- removed U3: MDBT50Q-1MV2, RF_Module:Raytac_MDBT50Q, symbol RF_Module:MDBT50Q-1MV2
- removed U4: BQ24074RGT, Package_DFN_QFN:VQFN-16-1EP_3x3mm_P0.5mm_EP1.6x1.6mm, symbol Battery_Management:BQ24074RGT
- added U: Beetle ESP32-C6, symbol beetle_esp32-c6:Beetle_ESP32-C6
- BT: renamed from BT1; value Battery_Cell -> 3.7V Li-Po 1000mAh
- D: renamed from D1; value WS2812B -> WS2812D
- renumbered BZ1 to BZ
Connections:
- net VBAT: now reaches BT.1 (+)
- net VBAT: now also U.16 (BAT)
- net GND: now reaches BT.2 (-)
- net GND: now also BZ.2 (-), D.3 (VSS), U.1 (GND), U.15 (GND)
- net +3V3: now reaches D.1 (VDD)
- net +3V3: now also U.2 (3V3)
- net LED_DATA: now reaches D.4 (DIN)
- net LED_DATA: now also U.12 (GPIO16)
- net BUZZER_CTRL: now reaches BZ.1 (+)
- net BUZZER_CTRL: now also U.10 (GPIO20)
- no-connect marks 0 -> 11
Other:
- note added: "2026-07-18"
- note added: "Central Unit Hub v2"
- note added: "Components: DFRobot Beetle ESP32-C6 / 3.7V 1000mAh Li-Po Battery / LED Diffused 5mm RGB Programmable WS2812D / Buzzer 2-5V 30mA"
- note added: "v2: Components updated. Wiring added. Revisions may occur."
- note removed: "09-07-26"
- note removed: "1. Power Management Unit"
- note removed: "2. Computing Unit"
- note removed: "3. Output Unit"
- note removed: "Acoustic Status Indicator"
- note removed: "Addressable Visual Status Indicator"
- note removed: "Battery Charge Management Controller"
- note removed: "Central Unit Hub v1"
- note removed: "Power Source (Battery Cell)"
- note removed: "Primary Microcontroller Unit (MCU)"
- note removed: "Secondary Communication Module (BLE)"
- note removed: "v1: A prototyping schematic of the central unit hub. No wiring. Changes to modules may apply."
- moved on the sheet: BT, BZ, D
