File: hardware/peripheral-unit/peripheral-unit.kicad_sch (KiCad schematic)
At the start: 8 parts, among them J1 Conn_01x08, J2 Conn_01x03, J3 Conn_01x02, U1 ESP32-H2-MINI-1-H2, U2 TPS22860DBVR, U3 LP2985-3.3

Commit message: v1.5: Minor Fixes
Parts:
- BT: renamed from BT1; value Battery_Cell -> Li-SOCl2 19000 mAh Battery
- C: renamed from C1; value C_Polarized -> Capacitor
Connections:
- net at C.1: now also BT.1 (+), U3.1 (VIN)
- net GND: now reaches C.2
- net GND: now also BT.2 (-), U3.2 (GND)
Other:
- note added: "Components: Waveshare ESP32-H2-Zero / EVE Energy ER34615 D-size Li-SOCl2 19000mAh Battery / low-ESR Tantalum capacitor or Solid Polymer capacitor (470-1000μF & 6.3V or 10V)"
- note added: "v2: Components updated. Wiring added."
- note removed: "1. Power Management Unit"
- note removed: "2. Computing Unit"
- note removed: "3. Sensor Unit"
- note removed: "3.6V Li-SOCl2 Battery"
- note removed: "HPC Pulse Capacitor"
- note removed: "Network Microcontroller"
- note removed: "v1: A prototype of the peripheral unit. No wiring. Changes may apply."
- moved on the sheet: BT, C, J3, U3
